File: PCB/GCP-2.kicad_pcb (KiCad board)
At the start: 4 copper layers, 45.3 x 26 mm, 46 parts, among them J1 USB4105-GF-A-060, J2 GC 1, J3 GC 2, J4 GC 3, J5 GC 4, SW1 1TS026A-1000-0550, SW2 1TS026A-1000-0550, SW3 1TS026A-1000-0550, U1 RP2040, U2 GD25Q80EEIGR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

Commit message: Update
Parts:
- added R14: 10k, Resistor_SMD:R_0201_0603Metric, B.Cu at (204.6, 148.3)
- C2: value 2.2uF -> 6.8uF
- U3: value 3.3v Fixed -> XC6222; footprint hhl:HTSOP-J8 -> hhl:SOT-89-5
- moved U3 4.56 mm to (208.3, 146.8), turned to 0 degrees
- moved C3 4.22 mm to (212.6, 144.4)
- moved TP3 3.65 mm to (207.1, 147.6)
- moved D1 2.13 mm to (212.1, 147.4), turned to -90 degrees
- moved F1 0.30 mm to (214.2, 147.6), turned to 90 degrees
Connections:
- C3 pad 2: Net-(D1-K) -> VCC
- D1 pad 1: Net-(D1-K) -> VCC
- F1 pad 2: VCC -> +5V
- J1 pad A4_B9: VCC -> +5V
- J1 pad B4_A9: VCC -> +5V
- J2 pad 3: +5V -> VCC
- J3 pad 3: +5V -> VCC
- J4 pad 3: +5V -> VCC
- J5 pad 3: +5V -> VCC
- TP5 pad 1: VCC -> +5V
- U3 pad 1: +3V3 -> Net-(U3-CE)
- U3 pad 2: +3V3 -> GND
- U3 pad 3: GND -> unconnected-(U3-NC-Pad3)
- U3 pad 4: GND -> VCC
- U3 pad 5: Net-(D1-K) -> +3V3
Routing:
- net VCC: track 16.8 -> 26.8 mm, vias 2 -> 5
- net +5V: track 21.2 -> 13.3 mm, vias 4 -> 2
- net Net-(D1-K): track 6.36 -> 0.00 mm
- net +3V3: track 111.8 -> 115.8 mm, vias 12 -> 13
- net GND: track 92.3 -> 88.8 mm, vias 15 -> 16
- net Net-(U3-CE): track 0.00 -> 2.37 mm
- net Net-(D1-A): track 3.54 -> 2.26 mm
- added copper zone on In2.Cu, net VCC
- removed copper zone on In2.Cu, net +5V
