File: PCB/GCP-2.kicad_sch (KiCad schematic)
At the start: 46 parts, among them J1 USB4105-GF-A-060, J2 GC 1, J3 GC 2, J4 GC 3, J5 GC 4, SW1 1TS026A-1000-0550, SW2 1TS026A-1000-0550, SW3 1TS026A-1000-0550, U1 RP2040, U2 GD25Q80EEIGR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

Commit message: Update
Parts:
- removed U3: 3.3v Fixed, hhl:HTSOP-J8, symbol hhl:BD33HA5WEFJ
- added R14: 10k, Resistor_SMD:R_0201_0603Metric, symbol Device:R_Small
- added U3: XC6222, hhl:SOT-89-5, symbol hhl:XC6222B331PR-G
- C2: value 2.2uF -> 6.8uF
Connections:
- net +3V3: now also U3.5 (Vout)
- net +5V: now also F1.2, J1.A4_B9 (VBUS), J1.B4_A9 (VBUS), TP5.1; no longer J2.3 (5V), J3.3 (5V), J4.3 (5V), J5.3 (5V)
- net GND: now also U3.2 (GND)
- net VCC: now also C3.2, D1.1 (K), J2.3 (5V), J3.3 (5V), J4.3 (5V), J5.3 (5V), R14.2, U3.4 (Vin); no longer F1.2, J1.A4_B9 (VBUS), J1.B4_A9 (VBUS), TP5.1
- new net: R14.1, U3.1 (CE)
Other:
- moved on the sheet: C1, C2, C3, D1
